Commit message: Removed the code things in ros1.

File: ros1/src/simulation/march_simulation/obstacles/curb.xacro (robot description, xacro)
@@ -5,6 +5,6 @@
     </gazebo>
     <xacro:property name="parent_name" value="world"/>
-    <xacro:property name="step_height" default="0.090"/>
-    <xacro:property name="step_depth" default="2"/>
+    <xacro:property name="step_height" default="0.170"/>
+    <xacro:property name="step_depth" default="7"/>
     <xacro:property name="step_width" default="1.80"/>
     <xacro:property name="distance_to_origin" default="0.45"/>
