Commit message: Change load_yaml to xacro.load_yaml since load_yaml is deprecated

File: ros2/src/shared/march_description/urdf/march4.xacro (robot description, xacro)
@@ -35,5 +35,5 @@
     <xacro:property name="config_yaml_file"
                     value="properties/march4.yaml"/>
-    <xacro:property name="properties" value="${load_yaml(config_yaml_file)}"/>
+    <xacro:property name="properties" value="${xacro.load_yaml(config_yaml_file)}"/>
     <xacro:property name="joint_limits" value="${properties['joint_limits']}"/>
     <xacro:property name="safety_values"

File: ros2/src/shared/march_description/urdf/march6.xacro (robot description, xacro)
@@ -39,5 +39,5 @@
     <xacro:property name="config_yaml_file"
                     value="properties/march6.yaml"/>
-    <xacro:property name="properties" value="${load_yaml(config_yaml_file)}"/>
+    <xacro:property name="properties" value="${xacro.load_yaml(config_yaml_file)}"/>
     <xacro:property name="joint_limits" value="${properties['joint_limits']}"/>
     <xacro:property name="safety_values"

File: ros2/src/shared/march_description/urdf/test_joint_linear.xacro (robot description, xacro)
@@ -26,5 +26,5 @@
     <xacro:property name="config_yaml_file"
                     value="properties/test_joints.yaml"/>
-    <xacro:property name="properties" value="${load_yaml(config_yaml_file)}"/>
+    <xacro:property name="properties" value="${xacro.load_yaml(config_yaml_file)}"/>
     <xacro:property name="joint_limits" value="${properties['joint_limits']}"/>
     <xacro:property name="safety_values"

File: ros2/src/shared/march_description/urdf/test_joint_rotational.xacro (robot description, xacro)
@@ -21,5 +21,5 @@
     <xacro:property name="config_yaml_file"
                     value="properties/test_joints.yaml"/>
-    <xacro:property name="properties" value="${load_yaml(config_yaml_file)}"/>
+    <xacro:property name="properties" value="${xacro.load_yaml(config_yaml_file)}"/>
     <xacro:property name="joint_limits" value="${properties['joint_limits']}"/>
     <xacro:property name="safety_values"
