Commit message: Change origin of start position

File: ros2/src/shared/march_description/urdf/march6_three_cameras.xacro (robot description, xacro)
@@ -396,10 +396,10 @@
                        parent="upper_leg_right"
                        plugin="$(arg realsense_simulation)">
-        <origin xyz="-0.08 0.035 -0.05 " rpy="${0 * pi} ${61/180 * pi} ${pi}"/>
+        <origin xyz="-0.08 0.035 -0.025 " rpy="${0 * pi} ${61/180 * pi} ${pi}"/>
     </xacro:sensor_d435>
     <xacro:sensor_d435 name="camera_front_left" topics_ns="camera_front_left"
                        parent="upper_leg_left"
                        plugin="$(arg realsense_simulation)">
-        <origin xyz="-0.08 -0.035 -0.05 " rpy="${0 * pi} ${61/180 * pi} ${pi}"/>
+        <origin xyz="-0.08 -0.035 -0.025 " rpy="${0 * pi} ${61/180 * pi} ${pi}"/>
     </xacro:sensor_d435>
     <xacro:sensor_d435 name="camera_back" topics_ns="camera_back" parent="hip_aa_frame_right_side"

Commit message: Align cameras in xacro

File: ros2/src/shared/march_description/urdf/march6_three_cameras.xacro (robot description, xacro)
@@ -396,10 +396,10 @@
                        parent="upper_leg_right"
                        plugin="$(arg realsense_simulation)">
-        <origin xyz="-0.08 0.035 -0.05 " rpy="${0 * pi} ${61/180 * pi} ${pi}"/>
+        <origin xyz="-0.08 0.035 -0.05 " rpy="${0 * pi} ${53/180 * pi} ${pi}"/>
     </xacro:sensor_d435>
     <xacro:sensor_d435 name="camera_front_left" topics_ns="camera_front_left"
                        parent="upper_leg_left"
                        plugin="$(arg realsense_simulation)">
-        <origin xyz="-0.08 -0.035 -0.05 " rpy="${0 * pi} ${61/180 * pi} ${pi}"/>
+        <origin xyz="-0.08 -0.045 -0.05 " rpy="${0 * pi} ${61/180 * pi} ${pi}"/>
     </xacro:sensor_d435>
     <xacro:sensor_d435 name="camera_back" topics_ns="camera_back" parent="hip_aa_frame_right_side"

Commit message: Make cameras vertical in urdf

File: ros2/src/shared/march_description/urdf/march6_three_cameras.xacro (robot description, xacro)
@@ -396,10 +396,10 @@
                        parent="upper_leg_right"
                        plugin="$(arg realsense_simulation)">
-        <origin xyz="-0.08 0.035 -0.05 " rpy="${0 * pi} ${53/180 * pi} ${pi}"/>
+        <origin xyz="-0.12 0.050 -0.015 " rpy="${-90/180 * pi} ${61/180 * pi} ${1*pi}"/>
     </xacro:sensor_d435>
     <xacro:sensor_d435 name="camera_front_left" topics_ns="camera_front_left"
                        parent="upper_leg_left"
                        plugin="$(arg realsense_simulation)">
-        <origin xyz="-0.08 -0.045 -0.05 " rpy="${0 * pi} ${61/180 * pi} ${pi}"/>
+        <origin xyz="-0.12 -0.035 -0.015 " rpy="${-90/180 * pi} ${61/180 * pi} ${1*pi}"/>
     </xacro:sensor_d435>
     <xacro:sensor_d435 name="camera_back" topics_ns="camera_back" parent="hip_aa_frame_right_side"

Commit message: Update urdf for new camera orientation

File: ros2/src/shared/march_description/urdf/march6_three_cameras.xacro (robot description, xacro)
@@ -396,10 +396,10 @@
                        parent="upper_leg_right"
                        plugin="$(arg realsense_simulation)">
-        <origin xyz="-0.08 0.035 -0.05 " rpy="${0 * pi} ${53/180 * pi} ${pi}"/>
+        <origin xyz="-0.12 0.050 -0.015 " rpy="${-90/180 * pi} ${53/180 * pi} ${1*pi}"/>
     </xacro:sensor_d435>
     <xacro:sensor_d435 name="camera_front_left" topics_ns="camera_front_left"
                        parent="upper_leg_left"
                        plugin="$(arg realsense_simulation)">
-        <origin xyz="-0.08 -0.045 -0.05 " rpy="${0 * pi} ${61/180 * pi} ${pi}"/>
+        <origin xyz="-0.12 -0.035 -0.015 " rpy="${-90/180 * pi} ${61/180 * pi} ${1*pi}"/>
     </xacro:sensor_d435>
     <xacro:sensor_d435 name="camera_back" topics_ns="camera_back" parent="hip_aa_frame_right_side"
