Commit message: Edit the copied march6 xacro to show the march7 xacro with correct visuals.

File: ros2/src/shared/march_description/urdf/march7.xacro (robot description, xacro)
@@ -38,5 +38,5 @@
     <!-- Add yaml files with properties -->
     <xacro:property name="config_yaml_file"
-                    value="properties/march6.yaml"/>
+                    value="properties/march7.yaml"/>
     <xacro:property name="properties" value="${load_yaml(config_yaml_file)}"/>
     <xacro:property name="joint_limits" value="${properties['joint_limits']}"/>
@@ -128,5 +128,5 @@
     <xacro:include filename="march.gazebo"/>
     <material name="visuals_material">
-        <color rgba="0.163 0.476 0.718 1"/>
+        <color rgba="1.0 1.0 1.0 1"/>
     </material>
     <!-- Used for fixing robot to Gazebo 'base_link' -->
@@ -138,7 +138,7 @@
                       length="${hip_base_height}"
                       direction="y"
-                      visual_origin="${hip_aa_frame_width} ${-width/2} ${-width/2}"
+                      visual_origin="0 0 0"
                       collision_origin="0 0 0"
-                      mesh="march6/HipBase.stl"
+                      mesh="march7/HipBase.stl"
                       com="${hip_base_com_x} ${hip_base_com_y} ${hip_base_com_z}"
                       mass="${dimensions['hip_base']['mass']}"
@@ -154,6 +154,6 @@
                       direction="y"
                       collision_origin="0 ${-hip_aa_frame_height/2} 0"
-                      visual_origin="${width/2} ${width/2 - 0.032} ${-width}"
-                      mesh="march6/HipLeft.stl"
+                      visual_origin="0 0 0"
+                      mesh="march7/HipLeft.stl"
                       visual_rpy="0 0 0"
     />
@@ -174,9 +174,10 @@
                       direction="z"
                       collision_origin="0 0 ${-upper_leg_height/2}"
-                      visual_origin="-0.01 -0.032 ${-upper_leg_height - width - 0.02}"
-                      mesh="march6/UpperLegLeft.stl"
+                      visual_origin="0 0 0"
+                      mesh="march7/UpperLegLeft.stl"
                       com="${upper_leg_com_x} ${-upper_leg_com_y} ${upper_leg_com_z}"
                       mass="${upper_leg_mass}"
                       inertia="${inertia['upper_leg']}"
+                      visual_rpy="0 0 0"
     />
     <xacro:frame_part name="lower_leg_left"
@@ -185,9 +186,10 @@
                       direction="z"
                       collision_origin="0 0 ${-lower_leg_height/2}"
-                      visual_origin="${width/2-0.02} -0.032 ${-lower_leg_height-width/2 - 0.01}"
-                      mesh="march6/LowerLegLeft.stl"
+                      visual_origin="0 0 0"
+                      mesh="march7/LowerLegLeft.stl"
                       com="${lower_leg_com_x} ${-lower_leg_com_y} ${lower_leg_com_z}"
                       mass="${lower_leg_mass}"
                       inertia="${inertia['lower_leg']}"
+                      visual_rpy="0 0 0"
     />
 <!-- Left Foot -->
@@ -196,8 +198,8 @@
                       length="${ankle_plate_height}"
                       direction="z"
-                      mesh="march6/FootLeft.stl"
-                      visual_origin="${-foot_height_forward+0.005} ${-ankle_plate_offset+knee_offset-width/2 - 0.02} ${-ankle_plate_height-width+0.01}"
+                      mesh="march7/FootLeft.stl"
+                      visual_origin="0 0 0"
                       collision_origin="0 0 ${-ankle_plate_height/2}"
-                      visual_rpy="0 0 ${pi}"
+                      visual_rpy="0 0 0"
     />
     <xacro:frame_part name="foot_left"
@@ -215,8 +217,8 @@
                       direction="y"
                       length="${hip_aa_frame_height}"
-                      visual_origin="${-width/2-hip_aa_frame_width - 0.007} ${-width/2 + 0.032} ${-width}"
+                      visual_origin="0 0 0"
                       collision_origin="0 ${hip_aa_frame_height/2} 0"
-                      mesh="march6/HipRight.stl"
-                      visual_rpy="0 0 ${pi}"
+                      mesh="march7/HipRight.stl"
+                      visual_rpy="0 0 0"
     />
     <xacro:frame_part name="hip_aa_frame_right_front"
@@ -235,6 +237,6 @@
                       length="${upper_leg_height}"
                       collision_origin="0 0 ${-upper_leg_height/2}"
-                      visual_origin="-0.01 0.032 ${-upper_leg_height - width - 0.02}"
-                      mesh="march6/UpperLegRight.stl"
+                      visual_origin="0 0 0"
+                      mesh="march7/UpperLegRight.stl"
                       com="${upper_leg_com_x} ${upper_leg_com_y} ${upper_leg_com_z}"
                       inertia="${inertia['upper_leg']}"
@@ -246,6 +248,6 @@
                       length="${lower_leg_height}"
                       direction="z"
-                      visual_origin="${width/2-0.025} 0.032 ${-lower_leg_height-width/2-0.01}"
-                      mesh="march6/LowerLegRight.stl"
+                      visual_origin="0 0 0"
+                      mesh="march7/LowerLegRight.stl"
                       com="${lower_leg_com_x} ${lower_leg_com_y} ${lower_leg_com_z}"
                       mass="${lower_leg_mass}"
@@ -259,6 +261,6 @@
                       length="${ankle_plate_height}"
                       direction="z"
-                      mesh="march6/FootRight.stl"
-                      visual_origin="0 ${ankle_plate_offset-knee_offset+width/2 + 0.02} ${-ankle_plate_height-width+0.01}"
+                      mesh="march7/FootRight.stl"
+                      visual_origin="0 0 0"
                       collision_origin="0 0 ${-ankle_plate_height/2}"
                       visual_rpy="0 0 0"
@@ -393,7 +395,7 @@
     </joint>
     <xacro:include filename="camera/_d435.urdf.xacro"/>
-    <xacro:sensor_d435 name="camera_back" topics_ns="camera_back" parent="hip_aa_frame_right_side"
+    <xacro:sensor_d435 name="camera_right" topics_ns="camera_back" parent="upper_leg_right"
                        plugin="$(arg realsense_simulation)">
-        <origin xyz="0 0.06725 0" rpy="0 ${75/180 * pi} 0"/>
+        <origin xyz="0.1 0 0" rpy="0 ${75/180 * pi} 0"/>
     </xacro:sensor_d435>
     <xacro:sensor_d435 name="camera_front" topics_ns="camera_front"

Commit message: Imrove collision object of the feet.

File: ros2/src/shared/march_description/urdf/march7.xacro (robot description, xacro)
@@ -87,4 +87,6 @@
     <xacro:property name="ankle_plate_offset"
                     value="${dimensions['ankle_plate']['offset']}"/>
+    <xacro:property name="ankle_plate_collision_offset"
+                value="${dimensions['ankle_plate']['collision_offset']}"/>
     <xacro:property name="foot_height_forward"
                     value="${dimensions['foot']['height_forward']}"/>
@@ -200,5 +202,5 @@
                       mesh="march7/FootLeft.stl"
                       visual_origin="0 0 0"
-                      collision_origin="0 0 ${-ankle_plate_height/2}"
+                      collision_origin="0 ${ankle_plate_collision_offset} ${-ankle_plate_height/2}"
                       visual_rpy="0 0 0"
     />
@@ -263,5 +265,5 @@
                       mesh="march7/FootRight.stl"
                       visual_origin="0 0 0"
-                      collision_origin="0 0 ${-ankle_plate_height/2}"
+                      collision_origin="0 ${-ankle_plate_collision_offset} ${-ankle_plate_height/2}"
                       visual_rpy="0 0 0"
     />
@@ -342,5 +344,5 @@
         <parent link="ankle_plate_left"/>
         <child link="foot_left"/>
-        <origin xyz="0 0 ${-ankle_plate_height-width/2}" rpy="0 0 0"/>
+        <origin xyz="0 ${ankle_plate_collision_offset} ${-ankle_plate_height-width/2}" rpy="0 0 0"/>
     </joint>
     <xacro:march_configurable_joint
@@ -392,5 +394,5 @@
         <parent link="ankle_plate_right"/>
         <child link="foot_right"/>
-        <origin xyz="0 0 ${-ankle_plate_height-width/2}" rpy="0 0 0"/>
+        <origin xyz="0 ${-ankle_plate_collision_offset} ${-ankle_plate_height-width/2}" rpy="0 0 0"/>
     </joint>
     <xacro:include filename="camera/_d435.urdf.xacro"/>
